Commit message: add kinova

File: examples/kinova_gen3/data/urdf/GEN3-7DOF-NOVISION_FOR_URDF_ARM_V12.urdf (robot description, URDF)
Before this commit: robot GEN3-7DOF-NOVISION_FOR_URDF_ARM_V12, 8 links, 7 joints
Links:
- link base_link: geometry collision mesh filename=/home/yurong/figaroh/models/others/robots/kinova_gen3/gen3/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; visual mesh filename=/home/yurong/figaroh/models/others/robots/kinova_gen3/gen3/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
- link bracelet_link: geometry collision mesh filename=/home/yurong/figaroh/models/others/robots/kinova_gen3/gen3/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; visual mesh filename=/home/yurong/figaroh/models/others/robots/kinova_gen3/gen3/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
- link forearm_link: geometry collision mesh filename=/home/yurong/figaroh/models/others/robots/kinova_gen3/gen3/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; visual mesh filename=/home/yurong/figaroh/models/others/robots/kinova_gen3/gen3/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
- link half_arm_1_link: geometry collision mesh filename=/home/yurong/figaroh/models/others/robots/kinova_gen3/gen3/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; visual mesh filename=/home/yurong/figaroh/models/others/robots/kinova_gen3/gen3/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
- link half_arm_2_link: geometry collision mesh filename=/home/yurong/figaroh/models/others/robots/kinova_gen3/gen3/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; visual mesh filename=/home/yurong/figaroh/models/others/robots/kinova_gen3/gen3/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
- link shoulder_link: geometry collision mesh filename=/home/yurong/figaroh/models/others/robots/kinova_gen3/gen3/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; visual mesh filename=/home/yurong/figaroh/models/others/robots/kinova_gen3/gen3/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
- link spherical_wrist_1_link: geometry collision mesh filename=/home/yurong/figaroh/models/others/robots/kinova_gen3/gen3/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; visual mesh filename=/home/yurong/figaroh/models/others/robots/kinova_gen3/gen3/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
- link spherical_wrist_2_link: geometry collision mesh filename=/home/yurong/figaroh/models/others/robots/kinova_gen3/gen3/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; visual mesh filename=/home/yurong/figaroh/models/others/robots/kinova_gen3/gen3/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

File: examples/kinova_gen3/data/urdf/robot.urdf (robot description, URDF)
Before this commit: robot gen3, 18 links, 17 joints
Links:
- link FT_adapter: geometry collision cylinder length=0.03 radius=0.0075
- link FT_sensor_mounting: geometry collision cylinder length=0.01 radius=0.0315; collision cylinder length=0.028 radius=0.035
- link base_link: geometry collision mesh filename=/home/yurong/figaroh/models/others/robots/kinova_gen3/gen3/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; visual mesh filename=/home/yurong/figaroh/models/others/robots/kinova_gen3/gen3/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
- link bracelet_link: geometry collision mesh filename=/home/yurong/figaroh/models/others/robots/kinova_gen3/gen3/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; visual mesh filename=/home/yurong/figaroh/models/others/robots/kinova_gen3/gen3/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
- link forearm_link: geometry collision mesh filename=/home/yurong/figaroh/models/others/robots/kinova_gen3/gen3/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; visual mesh filename=/home/yurong/figaroh/models/others/robots/kinova_gen3/gen3/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
- link half_arm_1_link: geometry collision mesh filename=/home/yurong/figaroh/models/others/robots/kinova_gen3/gen3/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; visual mesh filename=/home/yurong/figaroh/models/others/robots/kinova_gen3/gen3/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
- link half_arm_2_link: geometry collision mesh filename=/home/yurong/figaroh/models/others/robots/kinova_gen3/gen3/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; visual mesh filename=/home/yurong/figaroh/models/others/robots/kinova_gen3/gen3/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
- link shoulder_link: geometry collision mesh filename=/home/yurong/figaroh/models/others/robots/kinova_gen3/gen3/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; visual mesh filename=/home/yurong/figaroh/models/others/robots/kinova_gen3/gen3/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
- link spherical_wrist_1_link: geometry collision mesh filename=/home/yurong/figaroh/models/others/robots/kinova_gen3/gen3/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; visual mesh filename=/home/yurong/figaroh/models/others/robots/kinova_gen3/gen3/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
- link spherical_wrist_2_link: geometry collision mesh filename=/home/yurong/figaroh/models/others/robots/kinova_gen3/gen3/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; visual mesh filename=/home/yurong/figaroh/models/others/robots/kinova_gen3/gen3/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

File: examples/kinova_gen3/data/urdf/robot_updated.urdf (robot description, URDF)
Before this commit: robot gen3, 18 links, 17 joints
Links:
- link FT_adapter: geometry collision cylinder length=0.03 radius=0.0075
- link FT_sensor_mounting: geometry collision cylinder length=0.01 radius=0.0315; collision cylinder length=0.028 radius=0.035
- link base_link: geometry collision mesh filename=/home/yurong/figaroh/models/others/robots/kinova_gen3/gen3/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; visual mesh filename=/home/yurong/figaroh/models/others/robots/kinova_gen3/gen3/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
- link bracelet_link: mass 0.7228423358458282 -> 0.8313621489393325; geometry collision mesh filename=/home/yurong/figaroh/models/others/robots/kinova_gen3/gen3/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; visual mesh filename=/home/yurong/figaroh/models/others/robots/kinova_gen3/gen3/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
- link forearm_link: mass 0.9302000279332294 -> 0.994092576307687; geometry collision mesh filename=/home/yurong/figaroh/models/others/robots/kinova_gen3/gen3/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; visual mesh filename=/home/yurong/figaroh/models/others/robots/kinova_gen3/gen3/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
- link half_arm_1_link: mass 1.163600000000146 -> 1.031384648109728; geometry collision mesh filename=/home/yurong/figaroh/models/others/robots/kinova_gen3/gen3/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; visual mesh filename=/home/yurong/figaroh/models/others/robots/kinova_gen3/gen3/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
- link half_arm_2_link: mass 1.1635999999998636 -> 1.0814845354604532; geometry collision mesh filename=/home/yurong/figaroh/models/others/robots/kinova_gen3/gen3/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; visual mesh filename=/home/yurong/figaroh/models/others/robots/kinova_gen3/gen3/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
- link shoulder_link: mass 1.3772999720609305 -> 1.1746490194847434; geometry collision mesh filename=/home/yurong/figaroh/models/others/robots/kinova_gen3/gen3/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; visual mesh filename=/home/yurong/figaroh/models/others/robots/kinova_gen3/gen3/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
- link spherical_wrist_1_link: mass 0.6781000000057769 -> 0.8016193244823407; geometry collision mesh filename=/home/yurong/figaroh/models/others/robots/kinova_gen3/gen3/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; visual mesh filename=/home/yurong/figaroh/models/others/robots/kinova_gen3/gen3/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
- link spherical_wrist_2_link: mass 0.6781000000001965 -> 0.7992224156855354; geometry collision mesh filename=/home/yurong/figaroh/models/others/robots/kinova_gen3/gen3/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; visual mesh filename=/home/yurong/figaroh/models/others/robots/kinova_gen3/gen3/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
